Commit message: first commit

File: src/classic_nav_bringup/urdf/sentry_robot_sim.xacro (robot description, xacro)
@@ -237,6 +237,26 @@
     <origin xyz="$(arg xyz)" rpy="$(arg rpy)" />
   </xacro:mid360>
+    <!-- 深度相机仿真 -->
+  <xacro:include filename="$(find realsense_ros_gazebo)/xacro/depthcam.xacro"/>
+  <xacro:realsense_d435 sensor_name="d435_0" parent_link="base_link" rate="10">
+    <origin rpy="0 0 0" xyz="0 0 0.5"/>
+  </xacro:realsense_d435>
+  <xacro:realsense_d435 sensor_name="d435_1" parent_link="base_link" rate="10">
+    <origin rpy="0 0 ${pi/3}" xyz="0 0 0.5"/>
+  </xacro:realsense_d435>
+  <xacro:realsense_d435 sensor_name="d435_2" parent_link="base_link" rate="10">
+    <origin rpy="0 0 ${2*pi/3}" xyz="0 0 0.5"/>
+  </xacro:realsense_d435>
+  <xacro:realsense_d435 sensor_name="d435_3" parent_link="base_link" rate="10">
+    <origin rpy="0 0 ${pi}" xyz="0 0 0.5"/>
+  </xacro:realsense_d435>
+  <xacro:realsense_d435 sensor_name="d435_4" parent_link="base_link" rate="10">
+    <origin rpy="0 0 ${-2*pi/3}" xyz="0 0 0.5"/>
+  </xacro:realsense_d435>
+  <xacro:realsense_d435 sensor_name="d435_5" parent_link="base_link" rate="10">
+    <origin rpy="0 0 ${-pi/3}" xyz="0 0 0.5"/>
+  </xacro:realsense_d435>
   <!-- RGB camera仿真 -->
-  <link name="camera_link">
+  <!-- <link name="camera_link">
     <visual>
       <geometry>
@@ -259,8 +279,6 @@
     <child link="camera_link"/>
     <origin xyz="0.15 0 0.2" rpy="0 0 0"/>
-  </joint>
-  <joint name="camera_optical_joint" type="fixed">
-    <!-- these values have to be these values otherwise the gazebo camera image
-        won't be aligned properly with the frame it is supposedly originating from -->
+  </joint> -->
+  <!-- <joint name="camera_optical_joint" type="fixed">
     <origin xyz="0 0 0" rpy="${-pi/2} 0 ${-pi/2}"/>
     <parent link="camera_link"/>
@@ -268,6 +286,6 @@
   </joint>
   <link name="camera_link_optical">
-  </link>
-  <gazebo reference="camera_link">
+  </link> -->
+  <!-- <gazebo reference="camera_link">
     <sensor type="camera" name="camera_sensor">
       <update_rate>10.0</update_rate>
@@ -303,4 +321,4 @@
       </plugin>
     </sensor>
-  </gazebo>
+  </gazebo> -->
 </robot>
